Commit message: message

File: examples/rsc/ur5_description/urdf/finger_no1.urdf (robot description, URDF)
Before this commit: robot finger, 2 links, 1 joints
Links:
- removed link base
- added link left_inner_finger, mass 0.00724255346165745; collision box size=0.01 0.02 0.038; visual mesh filename=../meshes/ur5/visual/inner_finger_fine.STL
- added link left_inner_knuckle, mass 0.0110930853895903; collision box size=0.023 0.025 0.0135; visual mesh filename=../meshes/ur5/visual/inner_knuckle_fine.STL
- added link left_outer_finger, mass 0.0273093985570947; visual mesh filename=../meshes/ur5/visual/outer_finger_fine.STL
- added link left_outer_knuckle, mass 0.00684838849434396; visual mesh filename=../meshes/ur5/visual/outer_knuckle_fine.STL
- added link right_inner_finger, mass 0.00724255346165744; collision box size=0.01 0.02 0.038; visual mesh filename=../meshes/ur5/visual/inner_finger_fine.STL
- added link right_inner_knuckle, mass 0.0110930853895903; collision box size=0.023 0.025 0.0135; visual mesh filename=../meshes/ur5/visual/inner_knuckle_fine.STL
- added link right_outer_finger, mass 0.0273093985570947; visual mesh filename=../meshes/ur5/visual/outer_finger_fine.STL
- added link right_outer_knuckle, mass 0.00684838849401352; visual mesh filename=../meshes/ur5/visual/outer_knuckle_fine.STL
- link robotiq_85_base_link: mass 0.636951 -> 0.30915; geometry collision box size=0.03 0.015 0.095; visual mesh filename=../meshes/ur5/visual/robotiq_85_base_link_fine.STL
Joints:
- removed joint robotiq_85_base_joint
- added joint finger_joint: type revolute, parent robotiq_85_base_link, child left_outer_knuckle, origin xyz=0.0306011444260539 0 0.0627920162695395 rpy=0 0 0, axis 0 -1 0, limit lower=0 upper=0.725 effort=1000 velocity=2.0
- added joint left_inner_finger_joint: type revolute, parent left_inner_knuckle, child left_inner_finger, origin xyz=0.034585310861294 0 0.0454970193817975 rpy=0 0 0, axis 0 -1 0, limit lower=0 upper=0.8757 effort=1000 velocity=2.0, mimic joint=finger_joint multiplier=-1 offset=0
- added joint left_inner_knuckle_joint: type revolute, parent robotiq_85_base_link, child left_inner_knuckle, origin xyz=0.0127000000001501 0 0.0693074999999639 rpy=0 0 0, axis 0 -1 0, limit lower=0 upper=0.8757 effort=1000 velocity=2.0, mimic joint=finger_joint multiplier=1 offset=0
- added joint left_outer_finger_joint: type fixed, parent left_outer_knuckle, child left_outer_finger, origin xyz=0.0316910442266543 0 -0.00193396375724605 rpy=0 0 0, axis 0 -1 0
- added joint right_inner_finger_joint: type revolute, parent right_inner_knuckle, child right_inner_finger, origin xyz=0.0341060475457406 0 0.0458573878541688 rpy=0 0 0, axis 0 1 0, limit lower=0 upper=0.8757 effort=1000 velocity=2.0, mimic joint=finger_joint multiplier=1 offset=0
- added joint right_inner_knuckle_joint: type revolute, parent robotiq_85_base_link, child right_inner_knuckle, origin xyz=-0.0126999999998499 0 0.0693075000000361 rpy=0 0 3.14159265358979, axis 0 1 0, limit lower=0 upper=0.8757 effort=1000 velocity=2.0, mimic joint=finger_joint multiplier=-1 offset=0
- added joint right_outer_finger_joint: type fixed, parent right_outer_knuckle, child right_outer_finger, origin xyz=0.0317095909367246 0 -0.0016013564954687 rpy=0 0 0, axis 0 1 0
- added joint right_outer_knuckle_joint: type revolute, parent robotiq_85_base_link, child right_outer_knuckle, origin xyz=-0.0306011444258893 0 0.0627920162695395 rpy=0 0 3.14159265358979, axis 0 1 0, limit lower=0 upper=0.8757 effort=1000 velocity=2.0, mimic joint=finger_joint multiplier=-1 offset=0

File: examples/rsc/ur5_description/urdf/ur5.urdf.xacro (robot description, xacro)
@@ -71,13 +71,13 @@
       <visual>
         <geometry>
-          <mesh filename="package://ur5_description/meshes/ur5/visual/base.dae" />
-        </geometry>
-        <material name="LightGrey">
-          <color rgba="0.7 0.7 0.7 1.0"/>
-        </material>
-      </visual>
-      <collision>
-        <geometry>
-          <mesh filename="package://ur5_description/meshes/ur5/collision/base.stl" />
+          <mesh filename="../meshes/ur5/visual/base.dae" />
+        </geometry>
+        <material name="LightGrey">
+          <color rgba="0.7 0.7 0.7 1.0"/>
+        </material>
+      </visual>
+      <collision>
+        <geometry>
+          <mesh filename="../meshes/ur5/collision/base.stl" />
         </geometry>
       </collision>
